Commit message: fix shoulder and bow joints of bruce

File: resources/robots/bruce/urdf/bruce.urdf (robot description, URDF)
Before this commit: robot bruce, 17 links, 16 joints
Joints:
- joint elbow_pitch_l: type revolute -> fixed
- joint elbow_pitch_r: type revolute -> fixed
- joint shoulder_pitch_l: type revolute -> fixed
- joint shoulder_pitch_r: type revolute -> fixed
- joint shoulder_roll_l: type revolute -> fixed
- joint shoulder_roll_r: type revolute -> fixed
